File: microcontroller.kicad_sch (KiCad schematic)
At the start: 1 part, among them U2 STM32C031C6Tx

Commit message: progress
Parts:
- removed U2: STM32C031C6Tx, Package_QFP:LQFP-48_7x7mm_P0.5mm, symbol MCU_ST_STM32C0:STM32C031C6Tx
Changed lines of the file:
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@@
 	(generator_version "9.0")
 	(paper "A4")
-	(symbol
-		(lib_id "MCU_ST_STM32C0:STM32C031C6Tx")
-		(at 134.62 82.55 0)
-		(unit 1)
-		(exclude_from_sim no)
-		(in_bom yes)
-		(on_board yes)
-		(dnp no)
-		(fields_autoplaced yes)
-		(property "Reference" "U2"
-			(at 136.7633 31.75 0)
-			(effects
-				(font
-					(size 1.27 1.27)
-				)
-				(justify left)
-			)
-		)
-		(property "Value" "STM32C031C6Tx"
-			(at 136.7633 34.29 0)
-			(effects
-				(font
-					(size 1.27 1.27)
-				)
-				(justify left)
-			)
-		)
-		(property "Footprint" "Package_QFP:LQFP-48_7x7mm_P0.5mm"
-			(at 124.46 128.27 0)
-			(effects
-				(font
-					(size 1.27 1.27)
-				)
-				(justify right)
-				(hide yes)
-			)
-		)
-		(property "Datasheet" "https://www.st.com/resource/en/datasheet/stm32c031c6.pdf"
-			(at 134.62 82.55 0)
-			(effects
-				(font
-					(size 1.27 1.27)
-				)
-				(hide yes)
-			)
-		)
-		(property "Description" "STMicroelectronics Arm Cortex-M0+ MCU, 32KB flash, 12KB RAM, 48 MHz, 2.0-3.6V, 45 GPIO, LQFP48"
-			(at 134.62 82.55 0)
-			(effects
-				(font
-					(size 1.27 1.27)
-				)
-				(hide yes)
-			)
-		)
-		(pin "9"
-		)
-		(pin "10"
-		)
-		(pin "5"
-		)
-		(pin "40"
-		)
-		(pin "41"
-		)
-		(pin "38"
-		)
-		(pin "30"
-		)
-		(pin "39"
-		)
-		(pin "4"
-		)
-		(pin "8"
-		)
-		(pin "31"
-		)
-		(pin "6"
-		)
-		(pin "3"
-		)
-		(pin "7"
-		)
-		(pin "11"
-		)
-		(pin "13"
-		)
-		(pin "14"
-		)
-		(pin "16"
-		)
-		(pin "1"
-		)
-		(pin "2"
-		)
-		(pin "15"
-		)
-		(pin "12"
-		)
-		(pin "47"
-		)
-		(pin "33"
-		)
-		(pin "27"
-		)
-		(pin "32"
-		)
-		(pin "35"
-		)
-		(pin "36"
-		)
-		(pin "17"
-		)
-		(pin "28"
-		)
-		(pin "34"
-		)
-		(pin "19"
-		)
-		(pin "21"
-		)
-		(pin "45"
-		)
-		(pin "46"
-		)
-		(pin "48"
-		)
-		(pin "23"
-		)
-		(pin "25"
-		)
-		(pin "18"
-		)
-		(pin "26"
-		)
-		(pin "37"
-		)
-		(pin "29"
-		)
-		(pin "42"
-		)
-		(pin "20"
-		)
-		(pin "44"
-		)
-		(pin "43"
-		)
-		(pin "22"
-		)
-		(pin "24"
-		)
-		(instances
-			(project ""
-				(path "/81e8a54f-a6a6-4f78-985c-1dc7d6751007/10745524-5ba8-4327-b65c-e16bb0a1c7f6"
-					(reference "U2")
-					(unit 1)
-				)
-			)
-		)
-	)
 )
