File: Power_management.kicad_sch (KiCad schematic)
At the start: 0 parts

Commit message: updates
Other:
- removed sheet Microcontroller
- added sheet Buck Converter Stage (buck_converters.kicad_sch)
- sheet Cell Controller ports: added HS_SW_CP_EN, HS_SW_PCHG_EN, HS_SW_PMON_EN; removed none
- sheet Cell Monitor ports: added none; removed HS_SW_PACKDIV
- note added: "external commmunication from cell controller - i2c communication between cell monitor and controller so only 1 SMBUS connection is required"
Changed lines of the file:
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@@
 	(generator_version "9.0")
 	(paper "A4")
-	(text "REGOUT_AFE AT 3.3V?"
-		(exclude_from_sim no)
-		(at 137.414 45.974 0)
+	(text "external commmunication from cell controller - i2c \ncommunication between cell monitor and controller \nso only 1 SMBUS connection is required\n"
+		(exclude_from_sim no)
+		(at 255.778 28.448 0)
 		(effects
 			(font
@@
 		)
 	)
-	(text "HS_SW = HIGHSIDE SWITCHING - \nreferring to BQ76200PW high side switching driver"
-		(exclude_from_sim no)
-		(at 148.082 30.734 0)
+	(text "REGOUT_AFE AT 3.3V?"
+		(exclude_from_sim no)
+		(at 261.62 39.116 0)
 		(effects
 			(font
@@
 		)
 	)
+	(text "HS_SW = HIGHSIDE SWITCHING - \nreferring to BQ76200PW high side switching driver"
+		(exclude_from_sim no)
+		(at 256.54 17.526 0)
+		(effects
+			(font
+				(size 1.27 1.27)
+			)
+		)
+	)
 	(wire
 		(pts
@@
 	(wire
 		(pts
-			(xy 151.13 81.28) (xy 105.41 81.28)
+			(xy 105.41 45.72) (xy 158.75 45.72)
 		)
 		(stroke
@@
 	(wire
 		(pts
-			(xy 105.41 83.82) (xy 153.67 83.82)
+			(xy 105.41 48.26) (xy 158.75 48.26)
 		)
 		(stroke
@@
 	(wire
 		(pts
-			(xy 153.67 83.82) (xy 153.67 72.39)
+			(xy 142.24 68.58) (xy 158.75 68.58)
 		)
 		(stroke
@@
 	(wire
 		(pts
-			(xy 158.75 69.85) (xy 151.13 69.85)
+			(xy 142.24 71.12) (xy 158.75 71.12)
 		)
 		(stroke
@@
 	(wire
 		(pts
-			(xy 151.13 69.85) (xy 151.13 81.28)
-		)
-		(stroke
-			(width 0)
-			(type default)
-		)
-	)
-	(wire
-		(pts
 			(xy 105.41 59.69) (xy 114.3 59.69)
 		)
@@
 	(wire
 		(pts
-			(xy 153.67 72.39) (xy 158.75 72.39)
+			(xy 142.24 73.66) (xy 158.75 73.66)
 		)
 		(stroke
@@
 	)
 	(sheet
-		(at 101.6 111.76)
-		(size 29.21 22.86)
+		(at 81.28 124.46)
+		(size 34.29 16.51)
 		(exclude_from_sim no)
 		(in_bom yes)
@@
 			(color 0 0 0 0.0000)
 		)
-		(property "Sheetname" "Microcontroller"
-			(at 101.6 111.0484 0)
+		(property "Sheetname" "Buck Converter Stage"
+			(at 81.28 123.7484 0)
 			(effects
 				(font
@@
 			)
 		)
-		(property "Sheetfile" "microcontroller.kicad_sch"
-			(at 101.6 135.2046 0)
+		(property "Sheetfile" "buck_converters.kicad_sch"
+			(at 81.28 141.5546 0)
 			(effects
 				(font
@@
 	)
 	(sheet
-		(at 142.24 101.6)
+		(at 80.01 95.25)
 		(size 25.4 16.51)
 		(exclude_from_sim no)
@@
 		(fields_autoplaced yes)
 		(stroke
-			(width 0.1524)
+			(width 0.254)
 			(type solid)
+			(color 5 5 5 1)
 		)
 		(fill
-			(color 0 0 0 0.0000)
+			(color 255 203 223 1.0000)
 		)
 		(property "Sheetname" "USB Interface"
-			(at 142.24 100.8884 0)
+			(at 80.01 94.5384 0)
 			(effects
 				(font
@@
 		)
 		(property "Sheetfile" "usb_interface.kicad_sch"
-			(at 142.24 118.6946 0)
+			(at 80.01 112.3446 0)
 			(effects
 				(font
@@
 	)
 	(sheet
-		(at 68.58 107.95)
-		(size 24.13 10.16)
+		(at 114.3 95.25)
+		(size 27.94 16.51)
 		(exclude_from_sim no)
 		(in_bom yes)
@@
 		(fields_autoplaced yes)
 		(stroke
-			(width 0.1524)
+			(width 0.254)
 			(type solid)
+			(color 0 0 0 1)
 		)
 		(fill
-			(color 0 0 0 0.0000)
+			(color 255 203 223 1.0000)
 		)
 		(property "Sheetname" "Charger IC"
-			(at 68.58 107.2384 0)
+			(at 114.3 94.4876 0)
 			(effects
 				(font
@@
 		)
 		(property "Sheetfile" "charger_ic.kicad_sch"
-			(at 68.58 118.6946 0)
+			(at 114.3 112.3954 0)
 			(effects
 				(font
@@
 	)
 	(sheet
-		(at 80.01 52.07)
-		(size 25.4 33.02)
+		(at 80.01 43.18)
+		(size 25.4 41.91)
 		(exclude_from_sim no)
 		(in_bom yes)
@@
 		(fields_autoplaced yes)
 		(stroke
-			(width 0.1524)
+			(width 0.254)
 			(type solid)
+			(color 0 0 0 1)
 		)
 		(fill
-			(color 0 0 0 0.0000)
+			(color 255 203 223 1.0000)
 		)
 		(property "Sheetname" "Battery Pack"
-			(at 80.01 51.3584 0)
+			(at 80.01 42.4684 0)
 			(effects
 				(font
@@
 		)
 		(pin "BATT-" bidirectional
-			(at 105.41 83.82 0)
+			(at 105.41 48.26 0)
 			(effects
 				(font
@@
 		)
 		(pin "BATT+" bidirectional
-			(at 105.41 81.28 0)
+			(at 105.41 45.72 0)
 			(effects
 				(font
@@
 	)
 	(sheet
-		(at 158.75 52.07)
-		(size 35.56 27.94)
+		(at 158.75 44.45)
+		(size 35.56 35.56)
 		(exclude_from_sim no)
 		(in_bom yes)
@@
 		(fields_autoplaced yes)
 		(stroke
-			(width 0.1524)
+			(width 0.254)
 			(type solid)
+			(color 0 0 0 1)
 		)
 		(fill
-			(color 0 0 0 0.0000)
+			(color 255 203 223 1.0000)
 		)
 		(property "Sheetname" "Cell Controller"
-			(at 158.75 51.3584 0)
+			(at 158.75 43.7384 0)
 			(effects
 				(font
@@
 		)
 		(pin "BATT-" bidirectional
-			(at 158.75 72.39 180)
+			(at 158.75 48.26 180)
 			(effects
 				(font
@@
 		)
 		(pin "BATT+" bidirectional
-			(at 158.75 69.85 180)
+			(at 158.75 45.72 180)
 			(effects
 				(font
@@
 		(pin "REGOUT_AFE" bidirectional
 			(at 158.75 62.23 180)
+			(effects
+				(font
+					(size 1.27 1.27)
+				)
+				(justify left)
+			)
+		)
+		(pin "HS_SW_PCHG_EN" bidirectional
+			(at 158.75 71.12 180)
+			(effects
+				(font
+					(size 1.27 1.27)
+				)
+				(justify left)
+			)
+		)
+		(pin "HS_SW_CP_EN" bidirectional
+			(at 158.75 73.66 180)
+			(effects
+				(font
+					(size 1.27 1.27)
+				)
+				(justify left)
+			)
+		)
+		(pin "HS_SW_PMON_EN" bidirectional
+			(at 158.75 68.58 180)
 			(effects
 				(font
@@
 		(fields_autoplaced yes)
 		(stroke
-			(width 0.1524)
+			(width 0.254)
 			(type solid)
+			(color 0 0 0 1)
 		)
 		(fill
-			(color 0 0 0 0.0000)
+			(color 255 203 223 1.0000)
 		)
 		(property "Sheetname" "Cell Monitor"
@@
 		)
 		(pin "HS_SW_CP_EN" bidirectional
-			(at 142.24 76.2 0)
+			(at 142.24 73.66 0)
 			(effects
 				(font
@@
 		)
 		(pin "PACK-" bidirectional
-			(at 114.3 73.66 180)
+			(at 114.3 76.2 180)
 			(effects
 				(font
@@
 		)
 		(pin "HS_SW_PCHG_EN" bidirectional
-			(at 142.24 73.66 0)
+			(at 142.24 71.12 0)
 			(effects
 				(font
@@
 		)
 		(pin "PACK+" bidirectional
-			(at 114.3 71.12 180)
+			(at 114.3 73.66 180)
 			(effects
 				(font
@@
 		)
 		(pin "HS_SW_PMON_EN" bidirectional
-			(at 142.24 71.12 0)
-			(effects
-				(font
-					(size 1.27 1.27)
-				)
-				(justify right)
-			)
-		)
-		(pin "HS_SW_PACKDIV" bidirectional
 			(at 142.24 68.58 0)
 			(effects

Commit message: structural changes
Other:
- added sheet Power Distribution (pwr_distro.kicad_sch)
- sheet Buck Converter Stage ports: added 12V_Regout, 5V_Regout, PACK+, PACK-; removed none
- sheet Charger IC ports: added SCL_USBC, SDA_USBC; removed none
- sheet USB Interface ports: added SCL_USBC, SDA_USBC, USB_20V_BUS; removed none
- note added: "CHARGING"
- note added: "DISTRIBUTION"
- note added: "MONITORING"
- note added: "PMP22805 reference design - includes USB OTG for powering RADA ROCK 5B?"
- note added: "REGULATION"
