File: buck_converters.kicad_sch (KiCad schematic)
At the start: 44 parts, among them J12V1 Conn_01x02_Pin, J5V1 Conn_01x02_Pin, U6 SIC450ED-T1-GE3, U7 SIC450ED-T1-GE3

Commit message: structural changes
Parts:
- removed J12V1, J5V1, Jin1: Conn_01x02_Pin, symbol Connector:Conn_01x02_Pin
Connections:
- net +16V renamed PACK+
