File: pwr_distro.kicad_sch (KiCad schematic)
At the start: 3 parts, among them J1 USB_C_Receptacle, J12V1 Conn_01x02_Pin, J5V1 Conn_01x02_Pin

Commit message: refinements - moving battery pack off the PCB
Parts:
- added J4: USB3_A, symbol Connector:USB3_A
Changed lines of the file:
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@@
 	(rectangle
 		(start 44.45 18.415)
-		(end 236.855 95.885)
+		(end 142.24 95.885)
 		(stroke
 			(width 0)
@@
 		)
 	)
+	(rectangle
+		(start 147.32 17.78)
+		(end 245.11 95.25)
+		(stroke
+			(width 0)
+			(type default)
+		)
+		(fill
+			(type none)
+		)
+	)
+	(text_box "For radar"
+		(exclude_from_sim no)
+		(at 147.32 95.25 0)
+		(size 97.79 5.08)
+		(margins 0.9525 0.9525 0.9525 0.9525)
+		(stroke
+			(width 0)
+			(type solid)
+		)
+		(fill
+			(type none)
+		)
+		(effects
+			(font
+				(size 1.27 1.27)
+			)
+			(justify left top)
+		)
+	)
+	(text_box "3.3V distribution done through Raspberry PI outputs ??"
+		(exclude_from_sim no)
+		(at 38.1 158.75 0)
+		(size 97.79 5.08)
+		(margins 0.9525 0.9525 0.9525 0.9525)
+		(stroke
+			(width 0)
+			(type solid)
+		)
+		(fill
+			(type none)
+		)
+		(effects
+			(font
+				(size 1.27 1.27)
+			)
+			(justify left top)
+		)
+	)
 	(text_box "For RADA ROCK 5B"
 		(exclude_from_sim no)
 		(at 44.45 95.885 0)
-		(size 192.405 5.08)
+		(size 97.79 5.08)
 		(margins 0.9525 0.9525 0.9525 0.9525)
 		(stroke
@@
 					(unit 1)
 				)
+			)
+		)
+	)
+	(symbol
+		(lib_id "Connector:USB3_A")
+		(at 168.91 48.26 0)
+		(unit 1)
+		(exclude_from_sim no)
+		(in_bom yes)
+		(on_board yes)
+		(dnp no)
+		(fields_autoplaced yes)
+		(property "Reference" "J4"
+			(at 168.91 29.21 0)
+			(effects
+				(font
+					(size 1.27 1.27)
+				)
+			)
+		)
+		(property "Value" "USB3_A"
+			(at 168.91 31.75 0)
+			(effects
+				(font
+					(size 1.27 1.27)
+				)
+			)
+		)
+		(property "Footprint" ""
+			(at 172.72 45.72 0)
+			(effects
+				(font
+					(size 1.27 1.27)
+				)
+				(hide yes)
+			)
+		)
+		(property "Datasheet" "~"
+			(at 172.72 45.72 0)
+			(effects
+				(font
+					(size 1.27 1.27)
+				)
+				(hide yes)
+			)
+		)
+		(property "Description" "USB 3.0 A connector"
+			(at 168.91 48.26 0)
+			(effects
+				(font
+					(size 1.27 1.27)
+				)
+				(hide yes)
+			)
+		)
+		(pin "1"
+		)
+		(pin "4"
+		)
+		(pin "2"
+		)
+		(pin "3"
+		)
+		(pin "9"
+		)
+		(pin "7"
+		)
+		(pin "5"
+		)
+		(pin "8"
+		)
+		(pin "10"
+		)
+		(pin "6"
+		)
+		(instances
+			(project ""
+				(path "/81e8a54f-a6a6-4f78-985c-1dc7d6751007/47edc75a-ab5a-491b-b1f5-63eaaacac5fe"
+					(reference "J4")
+					(unit 1)
+				)
