File: Power_management.kicad_pcb (KiCad board)
At the start: 2 copper layers, 104.1 x 64.8 mm, 172 parts, among them J1 Screw_Terminal_01x02, J2 Conn_01x06, J3 Screw_Terminal_01x02, J4 Conn_01x03_Pin, J5 Conn_01x02_Pin, J6 USB_C_Receptacle, Q1 BUK7M67-60EX, Q2 BUK7M67-60EX, Q3 PMOS, Q4 NMOS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

Commit message: routing updates
Parts:
- J5: footprint Connector_PinHeader_2.54mm:PinHeader_1x02_P2.54mm_Vertical -> Connector_PinHeader_1.00mm:PinHeader_1x02_P1.00mm_Horizontal; moved to B.Cu
- moved R25 93.9 mm to (71.1, 67.3), turned to 0 degrees
- moved R24 87.1 mm to (71.1, 64.8), turned to 0 degrees
- moved R23 86.4 mm to (67.1, 61.0), turned to -90 degrees
- moved Q4 85.9 mm to (76.2, 64.8), turned to 0 degrees
- moved Q3 83.6 mm to (71.1, 61.0), turned to 0 degrees
- moved R22 81.9 mm to (80.0, 62.2), turned to -90 degrees
- moved R21 81.4 mm to (76.2, 61.0)
- moved C16 77.0 mm to (82.5, 62.2), turned to -90 degrees
- moved R27 74.8 mm to (62.2, 81.3)
- moved D2 73.4 mm to (67.6, 79.5), turned to -90 degrees
- moved J4 63.8 mm to (58.4, 73.2), turned to 0 degrees
- moved C17 59.5 mm to (75.5, 80.0), turned to 90 degrees
- moved R33 54.9 mm to (62.5, 73.2), turned to 180 degrees
- moved R34 54.6 mm to (62.5, 75.7), turned to 180 degrees
- moved D3 51.6 mm to (62.2, 71.1), turned to 180 degrees
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- renumbered SCL to TP3, SDA to TP4
Connections:
- net /Cell Monitor/HS_SW_PACKDIV renamed Net-(R17-Pad2)
- Q1 pad 4: /Cell Monitor/Top_cell_stack -> /Cell Monitor/CHG_GATE
- Q1 pad 5: /Cell Monitor/Top_cell_stack -> Net-(Q1-D)
- Q2 pad 1: /Cell Monitor/PACK+ -> Net-(Q1-D)
- Q2 pad 2: /Cell Monitor/PACK+ -> Net-(Q1-D)
- Q2 pad 3: /Cell Monitor/PACK+ -> Net-(Q1-D)
- Q2 pad 5: Net-(Q1-D) -> /Cell Monitor/PACK+
- Q5 pad 2: /Cell Monitor/Top_cell_stack -> Net-(Q5-G)
- R14 pad 2: /Cell Monitor/Top_cell_stack -> /Cell Monitor/CHG_GATE
- R41 pad 1: /Cell Monitor/Top_cell_stack -> /Charger IC/HIDRV1
- R41 pad 2: /Cell Monitor/Top_cell_stack -> Net-(Q5-G)
- U2 pad 16: /Cell Monitor/Top_cell_stack -> /Cell Monitor/CHG_GATE
Routing:
- net /Charger IC/SRN: track 0.00 -> 52.3 mm
- net /Charger IC/SRP: track 0.00 -> 50.5 mm
- net /Cell Monitor/Top_cell_stack: track 123.1 -> 157.8 mm
- net /Charger IC/HIDRV2: track 0.00 -> 32.9 mm
- net /Charger IC/LODRV2: track 0.00 -> 29.3 mm, vias 0 -> 2
- net /Cell Monitor/PACK-: track 28.5 -> 57.4 mm
- net /Charger IC/FB: track 0.00 -> 26.0 mm
- net /Charger IC/FBG: track 0.00 -> 21.9 mm
- net /Charger IC/HIDRV1: track 0.00 -> 20.9 mm, vias 0 -> 2
- net /Charger IC/POUT: track 0.00 -> 19.3 mm
- net /Cell Monitor/DSG: track 15.4 -> 0.00 mm
- net /Cell Monitor/CHG: track 15.1 -> 0.00 mm
- net +3V3: track 44.1 -> 59.2 mm
- net /Charger IC/REGN: track 16.7 -> 31.0 mm, vias 0 -> 2
- net /USB Interface/LDO_3V3: track 37.4 -> 50.2 mm
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Other:
- board text added: "short to reset BQ78350"

Commit message: compact routing- will address DRC errors
Parts:
- J5: footprint Connector_PinHeader_1.00mm:PinHeader_1x02_P1.00mm_Horizontal -> Connector_PinHeader_2.54mm:PinHeader_1x02_P2.54mm_Vertical
- moved R44 22.5 mm to (66.0, 38.1), turned to 90 degrees
- moved C18 19.8 mm to (89.7, 70.4), turned to 0 degrees
- moved R27 15.8 mm to (78.0, 81.2), turned to 90 degrees
- moved R10 14.2 mm to (67.3, 71.5), turned to 90 degrees
- moved R26 14.0 mm to (92.7, 71.6)
- moved TP2 13.7 mm to (95.0, 71.5)
- moved Cp3 12.8 mm to (38.1, 48.3)
- moved C8 12.7 mm to (62.2, 71.1)
- moved R9 12.7 mm to (59.7, 71.1)
- moved C1 12.7 mm to (54.6, 64.8)
- moved C11 12.7 mm to (58.4, 77.5)
- moved C2 12.7 mm to (54.6, 68.6)
- moved C3 12.7 mm to (54.6, 72.4)
- moved C4 12.7 mm to (54.6, 76.2)
- moved C5 12.7 mm to (54.6, 80.0)
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Routing:
- net +3V3: track 59.2 -> 192.0 mm, vias 2 -> 4
- net /Cell Controller/LED5: track 0.00 -> 44.8 mm, vias 0 -> 2
- net /Cell Controller/LED4: track 0.00 -> 42.8 mm, vias 0 -> 2
- net /Cell Controller/LED3: track 0.13 -> 41.0 mm, vias 0 -> 2
- net /Cell Controller/LED2: track 0.00 -> 39.5 mm, vias 0 -> 2
- net /Cell Controller/LED1: track 0.00 -> 38.7 mm, vias 0 -> 2
- net /Cell Monitor/DSG: track 0.00 -> 37.0 mm
- net /Cell Monitor/CHG: track 0.00 -> 36.8 mm
- net Net-(Q7-G): track 0.00 -> 28.5 mm
- net /Cell Controller/HS_SW_PCHG_EN: track 0.00 -> 26.1 mm, vias 0 -> 2
- net /Cell Monitor/ALERT_AFE: track 5.10 -> 30.1 mm, vias 0 -> 2
- net /Cell Controller/HS_SW_CP_EN: track 0.00 -> 23.4 mm
- net /Charger IC/HIDRV2: track 32.9 -> 10.2 mm
- net /Cell Controller/HS_SW_PMON_EN: track 0.00 -> 21.3 mm
- net /Cell Monitor/Top_cell_stack: track 157.8 -> 141.8 mm
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- added copper zone on F.Cu, net GND
Other:
- board size 104.1 x 64.8 mm -> 91.9 x 64.8 mm
