File: cell_controller.kicad_sch (KiCad schematic)
At the start: 30 parts, among them J2 Conn_01x03_Pin, Q1 NMOS, Q2 PMOS, U1 BQ78350DBT

Commit message: progress
Parts:
- removed D9: 599-2100-137F, LED_SMD:LED_1210_3225Metric, symbol Device:LED
- removed R17: 10, symbol Device:R
- added D10: LED, LED_SMD:LED_0805_2012Metric_Pad1.15x1.40mm_HandSolder, symbol Device:LED
- added R18: 700, symbol Device:R
- D2: value 599-2100-137F -> LED; footprint LED_SMD:LED_1210_3225Metric -> LED_SMD:LED_0805_2012Metric_Pad1.15x1.40mm_HandSolder
- D3, D4, D5, D6: footprint (none) -> LED_SMD:LED_0805_2012Metric_Pad1.15x1.40mm_HandSolder
- R10, R11, R12, R13, R5: value 10 -> 700
Connections:
- net REGOUT_AFE: now also R18.1
- new net: D10.2 (A), R18.2
Other:
- note added: "1.9V forward voltage drop at 2mA"
- note added: "APTD2012LCGCK LEDs"
