File: cell_monitor.kicad_sch (KiCad schematic)
At the start: 44 parts, among them Q8 BUK7M67-60EX, Q9 BUK7M67-60EX, SW1 SW_Push, U3 BQ76920PW, U5 BQ76200PW

Commit message: progress
Parts:
- renumbered Rsense to Rsense1
Other:
- note added: "75ppm rated to 4W"
- note removed: "75ppm"
