File: charger_ic.kicad_sch (KiCad schematic)
At the start: 0 parts

Commit message: starting usb pd charging
Parts:
- added C1: 4.7u, symbol Device:C
- added C2, C3, C4, C5: 0.01u, symbol Device:C
- added J1: USB_C_Receptacle, symbol Connector:USB_C_Receptacle
- added U5: TPS25730D, Package_DFN_QFN:Texas_REF0038A_WQFN-38-2EP_6x4mm_P0.4, symbol Interface_USB:TPS25730D
- added U6: BQ25798, Package_DFN_QFN:Texas_RQM0029A_VQFN-29_4x4mm_P0.4mm, symbol Battery_Management:BQ25798
- added U7: TVS2200DRV, Package_SON:WSON-6-1EP_2x2mm_P0.65mm_EP1x1.6mm, symbol Power_Protection:TVS2200DRV
Connections:
- new net: C1.1, C2.1, C3.1, C4.1, C5.1, J1.A4 (VBUS), J1.A9 (VBUS), J1.B4 (VBUS), J1.B9 (VBUS), U7.4 (IN), U7.5 (IN), U7.6 (IN)
- new net: U5.11 (GND), U5.12 (GND), U5.14 (GND), U5.16 (GND), U5.17 (GND), U5.31 (GND), U5.34 (GND), U5.39 (GND)
- new net: U6.2 (VBUS), U6.3 (VBUS)
- new net: U6.22 (BAT), U6.23 (BAT)
- new net GND: C1.2, C2.2, C3.2, C4.2, C5.2, J1.A1 (GND), J1.A12 (GND), J1.B1 (GND), J1.B12 (GND), J1.S1 (SHIELD), U7.1 (GND), U7.2 (GND), U7.3 (GND), U7.7 (GND)
- no-connect marks 0 -> 10

Commit message: usb pd charging
Parts:
- removed C1: 4.7u, symbol Device:C
- removed C2, C3, C4, C5: 0.01u, symbol Device:C
- removed J1: USB_C_Receptacle, symbol Connector:USB_C_Receptacle
- removed U5: TPS25730D, Package_DFN_QFN:Texas_REF0038A_WQFN-38-2EP_6x4mm_P0.4, symbol Interface_USB:TPS25730D
- removed U6: BQ25798, Package_DFN_QFN:Texas_RQM0029A_VQFN-29_4x4mm_P0.4mm, symbol Battery_Management:BQ25798
- removed U7: TVS2200DRV, Package_SON:WSON-6-1EP_2x2mm_P0.65mm_EP1x1.6mm, symbol Power_Protection:TVS2200DRV
- added U5: BQ25731RSNR, RSN0032B-IPC_A, symbol BQ25731RSNR:BQ25731RSNR
Connections:
- no-connect marks 10 -> 0

Commit message: progress
Parts:
- removed U5: BQ25731RSNR, RSN0032B-IPC_A, symbol BQ25731RSNR:BQ25731RSNR
Changed lines of the file:
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@@
 	(generator "eeschema")
 	(generator_version "9.0")
-	(paper "A4")
-	(symbol
-		(lib_id "BQ25731RSNR:BQ25731RSNR")
-		(at 115.57 43.18 0)
-		(unit 1)
-		(exclude_from_sim no)
-		(in_bom yes)
-		(on_board yes)
-		(dnp no)
-		(fields_autoplaced yes)
-		(property "Reference" "U5"
-			(at 142.24 33.02 0)
-			(effects
-				(font
-					(size 1.524 1.524)
-				)
-			)
-		)
-		(property "Value" "BQ25731RSNR"
-			(at 142.24 35.56 0)
-			(effects
-				(font
-					(size 1.524 1.524)
-				)
-			)
-		)
-		(property "Footprint" "RSN0032B-IPC_A"
-			(at 115.57 43.18 0)
-			(effects
-				(font
-					(size 1.27 1.27)
-					(italic yes)
-				)
-				(hide yes)
-			)
-		)
-		(property "Datasheet" "https://www.ti.com/lit/gpn/bq25731"
-			(at 115.57 43.18 0)
-			(effects
-				(font
-					(size 1.27 1.27)
-					(italic yes)
-				)
-				(hide yes)
-			)
-		)
-		(property "Description" ""
-			(at 115.57 43.18 0)
-			(effects
-				(font
-					(size 1.27 1.27)
-				)
-				(hide yes)
-			)
-		)
-		(pin "23"
-		)
-		(pin "21"
-		)
-		(pin "18"
-		)
-		(pin "20"
-		)
-		(pin "8"
-		)
-		(pin "9"
-		)
-		(pin "28"
-		)
-		(pin "24"
-		)
-		(pin "22"
-		)
-		(pin "19"
-		)
-		(pin "26"
-		)
-		(pin "17"
-		)
-		(pin "16"
-		)
-		(pin "2"
-		)
-		(pin "6"
-		)
-		(pin "11"
-		)
-		(pin "13"
-		)
-		(pin "3"
-		)
-		(pin "4"
-		)
-		(pin "15"
-		)
-		(pin "14"
-		)
-		(pin "12"
-		)
-		(pin "5"
-		)
-		(pin "25"
-		)
-		(pin "10"
-		)
-		(pin "33"
-		)
-		(pin "27"
-		)
-		(pin "29"
-		)
-		(pin "30"
-		)
-		(pin "31"
-		)
-		(pin "7"
-		)
-		(pin "32"
-		)
-		(pin "1"
-		)
-		(instances
-			(project ""
-				(path "/81e8a54f-a6a6-4f78-985c-1dc7d6751007/74145ec3-99f0-43b9-89a7-81e8f7fd18fe"
-					(reference "U5")
-					(unit 1)
-				)
-			)
-		)
-	)
+	(paper "A3")
 )

Commit message: structural changes
Parts:
- added U8: BQ25731RSNR, RSN0032B-IPC_A, symbol BQ25731:BQ25731RSNR
Connections:
- new net SCL_USBC: U8.13 (SCL)
- new net SDA_USBC: U8.12 (SDA)
Changed lines of the file:
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@@
 	(generator_version "9.0")
 	(paper "A3")
+	(wire
+		(pts
+			(xy 167.64 160.02) (xy 157.48 160.02)
+		)
+		(stroke
+			(width 0)
+			(type default)
+		)
+	)
+	(wire
+		(pts
+			(xy 167.64 165.1) (xy 157.48 165.1)
+		)
+		(stroke
+			(width 0)
+			(type default)
+		)
+	)
+	(hierarchical_label "SCL_USBC"
+		(shape input)
+		(at 157.48 160.02 180)
+		(effects
+			(font
+				(size 1.27 1.27)
+			)
+			(justify right)
+		)
+	)
+	(hierarchical_label "SDA_USBC"
+		(shape input)
+		(at 157.48 165.1 180)
+		(effects
+			(font
+				(size 1.27 1.27)
+			)
+			(justify right)
+		)
+	)
+	(symbol
+		(lib_id "BQ25731:BQ25731RSNR")
+		(at 167.64 91.44 0)
+		(unit 1)
+		(exclude_from_sim no)
+		(in_bom yes)
+		(on_board yes)
+		(dnp no)
+		(fields_autoplaced yes)
+		(property "Reference" "U8"
+			(at 194.31 81.28 0)
+			(effects
+				(font
+					(size 1.524 1.524)
+				)
+			)
+		)
+		(property "Value" "BQ25731RSNR"
+			(at 194.31 83.82 0)
+			(effects
+				(font
+					(size 1.524 1.524)
+				)
+			)
+		)
+		(property "Footprint" "RSN0032B-IPC_A"
+			(at 167.64 91.44 0)
+			(effects
+				(font
+					(size 1.27 1.27)
+					(italic yes)
+				)
+				(hide yes)
+			)
+		)
+		(property "Datasheet" "https://www.ti.com/lit/gpn/bq25731"
+			(at 167.64 91.44 0)
+			(effects
+				(font
+					(size 1.27 1.27)
+					(italic yes)
+				)
+				(hide yes)
+			)
+		)
+		(property "Description" ""
+			(at 167.64 91.44 0)
+			(effects
+				(font
+					(size 1.27 1.27)
+				)
+				(hide yes)
+			)
+		)
+		(pin "25"
+		)
+		(pin "11"
+		)
+		(pin "16"
+		)
+		(pin "21"
+		)
+		(pin "23"
+		)
+		(pin "20"
+		)
+		(pin "5"
+		)
+		(pin "19"
+		)
+		(pin "17"
+		)
+		(pin "28"
+		)
+		(pin "24"
+		)
+		(pin "1"
+		)
+		(pin "27"
+		)
+		(pin "33"
+		)
+		(pin "3"
+		)
+		(pin "15"
+		)
+		(pin "14"
+		)
+		(pin "31"
+		)
+		(pin "6"
+		)
+		(pin "4"
+		)
+		(pin "26"
+		)
+		(pin "22"
+		)
+		(pin "29"
+		)
+		(pin "9"
+		)
+		(pin "8"
+		)
+		(pin "10"
+		)
+		(pin "32"
+		)
+		(pin "30"
+		)
+		(pin "7"
+		)
+		(pin "18"
+		)
+		(pin "13"
+		)
+		(pin "12"
+		)
+		(pin "2"
+		)
+		(instances
+			(project ""
+				(path "/81e8a54f-a6a6-4f78-985c-1dc7d6751007/74145ec3-99f0-43b9-89a7-81e8f7fd18fe"
+					(reference "U8")
+					(unit 1)
+				)
+			)
+		)
+	)
 )

Commit message: adding charging stages finally
Parts:
- removed U8: BQ25731RSNR, RSN0032B-IPC_A, symbol BQ25731:BQ25731RSNR
- added C19, C20, C43, C54, C55, C57: 100nF 100V, symbol Device:C
- added C21: C_Polarized, symbol Device:C_Polarized
- added C22: C, symbol Device:C
- added C33: 100pF 100V, symbol Device:C
- added C34, C35: 100nF 25V, symbol Device:C
- added C36, C58: 4.7u 25V, symbol Device:C
- added C42, C56: 470nF 16V, symbol Device:C
- added D19, D20: V1FM10-M3/H, symbol Device:D_Schottky
- added L3: L, symbol Device:L
- added Q11, Q12, Q13, Q7: 45V 100A, symbol Simulation_SPICE:NMOS
- added R37: 1M, symbol Device:R
- added R47: 26.7k, symbol Device:R
- added R48: 36.5k, symbol Device:R
- added R49, R50, R51, R52: 10k, symbol Device:R
- added R74, R75: 3.3k, symbol Device:R
- added R76: 100k, symbol Device:R
- added R77: 249k 0.1%, symbol Device:R
- added R78: 22.9k, symbol Device:R
- added R79: 1.1, symbol Device:R
- added R80, R86: 5m, symbol Device:R
- added R81, R82, R85, R87: 10, symbol Device:R
- added R83, R84, R88, R89: 0, symbol Device:R
- added TP5: SDA Testpoint, symbol Connector:TestPoint
- added TP6: SCL Testpoint, symbol Connector:TestPoint
- added U8: BQ25756ERRVR, VQFN36_RRV_TEX, symbol BQ25756E:BQ25756ERRVR
Connections:
- new net: Q7.2 (G), R83.2
- new net: R74.2, TP5.1, U8.1 (SCL)
- new net: Q12.2 (G), R88.2
- new net: Q11.2 (G), R84.2
- new net: C33.1, R79.2
- new net: Q13.2 (G), R89.2
- new net: R75.2, TP6.1, U8.2 (SDA)
- new net *INT: R50.2, U8.3 (*INT)
- new net *PG: R49.2, U8.6 (*PG)
- new net +3V3: R49.1, R50.1, R51.1, R52.1, R74.1, R75.1
- new net ACN: C42.2, C54.1, R82.2, U8.29 (ACN)
- new net ACOV: C20.1, R47.2, R48.1
- new net ACP: C42.1, C43.1, R81.2, U8.30 (ACP)
- new net ACUV: C19.1, R37.2, R47.1
- new net BATT+: R77.2, R79.1, R85.1, R86.1
- new net BTST1: C34.1, D19.1 (K), U8.26 (BTST1)
- new net BTST2: C35.1, D20.1 (K), U8.20 (BTST2)
- new net FB: C33.2, R77.1, R78.1, U8.12 (FB)
- new net FBG: R78.2, U8.11 (FBG)
- new net FSW_SYNC: R76.1, U8.36 (FSW_SYNC)
- new net GND: C19.2, C20.2, C36.2, C43.2, C54.2, C55.2, C57.2, C58.2, Q12.3 (S), Q13.3 (S), R48.2, R76.2, U8.17 (PGND), U8.22 (PGND), U8.37 (EPAD), U8.7 (*CE)
- new net HIDRV1: R83.1
- new net HIDRV2: R84.1, U8.19 (HIDRV2)
- new net LODRV1: R88.1, U8.25 (LODRV1)
- new net LODRV2: R89.1, U8.21 (LODRV2)
- new net POUT: Q11.1 (D), R86.2, R87.1
- new net PPHV: R37.1, R80.1, R81.1
- new net REGN: C36.1, C58.1, D19.2 (A), D20.2 (A), U8.23 (DRV_SUP), U8.24 (REGN)
- new net SRN: C55.1, C56.1, R85.2, U8.13 (SRN)
- new net SRP: C56.2, C57.1, R87.2, U8.14 (SRP)
- new net STAT1: R51.2, U8.4 (STAT1)
- new net STAT2: R52.2, U8.5 (STAT2)
- new net SW1: C34.2, L3.1, Q12.1 (D), Q7.3 (S), U8.28 (SW1)
- new net SW2: C35.2, L3.2, Q11.3 (S), Q13.1 (D), U8.18 (SW2)
- new net VSYS: Q7.1 (D), R80.2, R82.1
Other:
- note added: "datasheet 9.2.1.2.2 for selection details"
- note added: "figure out where this is going to come from"

Commit message: finished charger schematic - still need to finalise usb
Parts:
- added C23, C26, C28, C30: 4.7uF 50V, symbol Device:C
- added C24, C27: 47uF 50V, symbol Device:C_Polarized
- added C25: 100nF 50V, symbol Device:C
- added C29: 68uF 35V, symbol Device:C_Polarized
- added J3: Conn_01x02_Pin, symbol Connector:Conn_01x02_Pin
- added R53: 25k, symbol Device:R
- added R54: 6.65k, symbol Device:R
- added R55: 3.61k, symbol Device:R
- added R56: 15.48k, symbol Device:R
- C21: value C_Polarized -> 47uF 35V
- C22: value C -> 100nF 50V
- L3: value L -> 10uH
Connections:
- net ACOV: now also U8.35 (ACOV)
- net ACUV: now also U8.34 (ACUV)
- net BATT+: now also C27.1, C28.1
- net GND: now also C21.2, C22.2, C23.2, C24.2, C25.2, C26.2, C27.2, C28.2, C29.2, C30.2, J3.2 (Pin_2), R53.2, R54.2, R56.2
- net HIDRV1: now also U8.27 (HIDRV1)
- net POUT: now also C24.1, C25.1, C26.1
- net PPHV: now also U8.32 (VAC), U8.33 (VAC), C29.1, C30.1
- net REGN: now also R55.1
- net VSYS: now also C21.1, C22.1, C23.1
- net ILIM_HIZ: now reaches U8.10 (ILIM_HIZ)
- net ILIM_HIZ: now also R54.1
- net TS: now reaches U8.8 (TS)
- net TS: now also J3.1 (Pin_1), R55.2, R56.1
- net ICHG: now reaches U8.9 (ICHG)
- net ICHG: now also R53.1
Other:
- moved on the sheet: C21, C22, R49, R50, R51, R52, R74, R75, TP5, TP6
