File: usb_interface.kicad_sch (KiCad schematic)
At the start: 7 parts, among them J1 USB_C_Receptacle, U7 TVS2200DRV

Commit message: progress
Parts:
- added C1: 4.7u, symbol Device:C
- added C2, C3: 330p, symbol Device:C
- added R6, R7, R8: 10k, symbol Device:R
- added U2: TPS25730D, Package_DFN_QFN:Texas_REF0038A_WQFN-38-2EP_6x4mm_P0.4, symbol Interface_USB:TPS25730D
- J15: renamed from J1; footprint (none) -> Connector_USB:USB_C_Receptacle_GCT_USB4105-xx-A_16P_TopMnt_Horizontal
- renumbered C1 to C45, C2 to C46, C3 to C47, C4 to C48, C5 to C49, U7 to U4
Connections:
- net GND: now also C1.2, C2.2, C3.2, R6.2, R7.2, R8.2
- net at C45.1, C46.1, C47.1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: now also U2.23 (VBUS_IN), U2.32 (VBUS)
- net at J15.A5 (CC1): now also C2.1, U2.28 (CC1)
- net at J15.B5 (CC2): now also C3.1, U2.29 (CC2)
- new net: R6.1, U2.26 (RESERVED)
- new net: R8.1, U2.36 (RESERVED)
- new net: U2.11 (GND), U2.12 (GND), U2.14 (GND), U2.16 (GND), U2.17 (GND), U2.31 (GND), U2.34 (GND), U2.39 (GND)
- new net: R7.1, U2.27 (RESERVED)
- new net: C1.1, U2.4 (LDO_1V5)
- new net USB_20V_BUS: U2.20 (PPHV)
Other:
- moved on the sheet: U4

Commit message: structural changes
Parts:
- added C14, C15, C18: 10u, symbol Device:C
- added C16, C17: 22u, symbol Device:C
- added F3: 5A, symbol Device:Fuse
- added R23, R24: 10k, symbol Device:R
- added R30: 190k, symbol Device:R
- added R31: 9.5k, symbol Device:R
- added R41: 162k, symbol Device:R
- added R42: 38k, symbol Device:R
- added R43: 9.4k, symbol Device:R
- added R44: 191k, symbol Device:R
- added R45: 198.2k, symbol Device:R
- added R46: 2.28k, symbol Device:R
Connections:
- net GND: now also C14.2, C15.2, C16.2, C17.2, C18.2, R31.2, R42.2, R44.2, R46.2
- net USB_20V_BUS: now also C16.1, C17.1, C18.1
- net CC1: now reaches C2.1, J15.A5 (CC1), U2.28 (CC1)
- net RES_26: now reaches R6.1, U2.26 (RESERVED)
- net at C45.1, C46.1, C47.1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: now also F3.1; no longer U2.23 (VBUS_IN), U2.32 (VBUS)
- net RES_28: now reaches R8.1, U2.36 (RESERVED)
- net LDO_3V3: now reaches U2.1 (LDO_3V3)
- net LDO_3V3: now also C14.1, R23.1, R24.1, R30.1, R41.1, R43.1, R45.1
- net DRAIN: now reaches U2.15 (DRAIN)
- net DRAIN: now also U2.30 (DRAIN), U2.40 (DRAIN)
- net ADCIN1: now reaches U2.2 (ADCIN1)
- net ADCIN1: now also R45.2, R46.1
- net RES_27: now reaches R7.1, U2.27 (RESERVED)
- net CC2: now reaches C3.1, J15.B5 (CC2), U2.29 (CC2)
- net ADCIN2: now reaches U2.3 (ADCIN2)
- net ADCIN2: now also R43.2, R44.1
- net LDO_1V5: now reaches C1.1, U2.4 (LDO_1V5)
- net ADCIN3: now reaches U2.5 (ADCIN3)
- net ADCIN3: now also R41.2, R42.1
- net ADCIN4: now reaches U2.7 (ADCIN4)
- net ADCIN4: now also R30.2, R31.1
- net SDA_USBC: now reaches U2.8 (I2Ct_SDA)
- net SDA_USBC: now also R23.2
- net SCL_USBC: now reaches U2.9 (I2Ct_SCL)
- net SCL_USBC: now also R24.2
- new net VBUS: F3.2, U2.23 (VBUS_IN), U2.32 (VBUS)
- new net VIN_3V3: C15.1
- no-connect marks 10 -> 14
Other:
- note added: "Charging system will only work with USB C PD enabled chargers"
- note added: "Configured for 20V @ 3A as TPS25730D datasheet example - page 42"
- note added: "LED to indicate this is high?"
- note added: "tie together with large copper plane - part of 3A path so likely to get HOT"
- moved on the sheet: C1, C2, C3, C45, C46, C47, C48, C49, J15, U2, U4

Commit message: adding charging stages finally
Connections:
- net USB_20V_BUS renamed PPHV
Other:
- note added: "660uA from LDO_3V3"
- note added: "66uA from LDO_3V3"
- note added: "max 1mA draw - do not overload - already at 726uA dont make external connections"
Changed lines of the file:
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@@
+		)
+	)
+	(text "max 1mA draw - do not overload - already at 726uA dont make external connections"
+		(exclude_from_sim no)
+		(at 60.198 110.236 0)
+		(effects
+			(font
+				(size 1.27 1.27)
+			)
 		)
 	)
@@
 				(size 1.27 1.27)
 				(color 255 83 131 1)
+			)
+		)
+	)
+	(text "66uA from LDO_3V3"
+		(exclude_from_sim no)
+		(at 260.604 45.212 0)
+		(effects
+			(font
+				(size 1.27 1.27)
+			)
+		)
+	)
+	(text "660uA from LDO_3V3"
+		(exclude_from_sim no)
+		(at 178.054 37.846 0)
+		(effects
+			(font
+				(size 1.27 1.27)
 			)
 		)
@@
 		)
 	)
-	(hierarchical_label "USB_20V_BUS"
+	(hierarchical_label "PPHV"
 		(shape input)
 		(at 267.97 99.06 0)

Commit message: finished charger schematic - still need to finalise usb
Parts:
- added C31: 4.7u, symbol Device:C
- added R57: 1k, symbol Device:R
- added R58: 10k, symbol Device:R
Connections:
- net GND: now also C31.2, R58.2
- net LDO_3V3: now also R57.1
- net VBUS: now also C31.1
- net at U2.18 (~{FAULT_IN}): now also R57.2, R58.1
- no-connect marks 14 -> 19
Other:
- note added: "unused open drain outputs"
